File: terasic-adapter.kicad_pcb (KiCad board)
At the start: 2 copper layers, 68.6 x 106.8 mm, 21 parts, among them J1 Conn_02x20_Odd_Even, J2 Conn_02x05_Odd_Even, J3 Conn_02x05_Odd_Even, J4 Conn_02x05_Odd_Even, J5 Conn_02x05_Odd_Even, U1 TPS793333-EP, U2 4066

Commit message: fix part spelling for TPS79333-EP
Fixed in upstream https://github.com/kicad/kicad-symbols
by commit 5da4de5bcafbec757f83fc1941268a7594b1ae7c
(fix part spelling for TPS79333-EP)

Signed-off-by: Antony Pavlov <antonynpavlov@gmail.com>
Parts:
- U1: value TPS793333-EP -> TPS79333-EP
Changed lines of the file:
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@@
       (effects (font (size 1 1) (thickness 0.15)))
     )
-    (fp_text value TPS793333-EP (at 0 2.9) (layer F.Fab) hide
+    (fp_text value TPS79333-EP (at 0 2.9) (layer F.Fab) hide
       (effects (font (size 1 1) (thickness 0.15)))
     )
